Commit message: Added new global <xacro:property> "actor_bone_scaling_map" to represent list of pairs of names of different "bone" links used in <actor> .dae skeleton, mapped to X/Y/Z scaling factors (as copied from original example.world used for CollisionActorPlugin example in servicesim_competition package).
New <xacro:macro> "make_one_scaling" to generate SDF block expected by CollisionActorPlugin code (for scaling factor mapped values), as well as now for new TrajectoryActorExtendedPlugin code.

New <xacro:macro> "loop_through_scaling" to (non-destructively) loop through list of values in "actor_bone_scaling_map" global <xacro:property>, to generate full set of <scaling> elements expected by CollisionActorPlugin & TrajectoryActorExtendedPlugin code.

Updated <xacro:macro> "make_one_actor_traj_model" to add new optional input parameter "bScaleSkel4Collision", so as to enable runtime switching between SDF blocks for supporting extended logic of TrajectoryActorExtendedPlugin, which incorporates (modified) CollisionActorPlugin logic into the original TrajectoryActorPlugin.

File: worlds/lib_actor.world.xacro (robot description, xacro)
@@ -1,4 +1,26 @@
 <?xml version="1.0" ?>
 <robot xmlns:xacro="http://www.ros.org/wiki/xacro">
+<xacro:property name="actor_bone_scaling_map" value="${[
+	[ 'LHipJoint_LeftUpLeg',    [ 0.01, 0.001, 0.001 ] ],
+	[ 'LeftUpLeg_LeftLeg',      [ 8.0, 8.0, 1.0 ] ],
+	[ 'LeftLeg_LeftFoot',       [ 8.0, 8.0, 1.0 ] ],
+	[ 'LeftFoot_LeftToeBase',   [ 4.0, 4.0, 1.5 ] ],
+	[ 'RHipJoint_RightUpLeg',   [ 0.01, 0.001, 0.001 ] ],
+	[ 'RightUpLeg_RightLeg',    [ 8.0, 8.0, 1.0 ] ],
+	[ 'RightLeg_RightFoot',     [ 8.0, 8.0, 1.0 ] ],
+	[ 'RightFoot_RightToeBase', [ 4.0, 4.0, 1.5 ] ],
+	[ 'LowerBack_Spine', [ 12.0, 20.0, 5.0 ], '0.05 0 0 0 -0.2 0' ],
+	[ 'Spine_Spine1',           [ 0.01, 0.001, 0.001 ] ],
+	[ 'Neck_Neck1',             [ 0.01, 0.001, 0.001 ] ],
+	[ 'Neck1_Head',             [ 5.0, 5.0, 3.0 ] ],
+	[ 'LeftShoulder_LeftArm',   [ 0.01, 0.001, 0.001 ] ],
+	[ 'LeftArm_LeftForeArm',    [ 5.0, 5.0, 1.0 ] ],
+	[ 'LeftForeArm_LeftHand',   [ 5.0, 5.0, 1.0 ] ],
+	[ 'LeftFingerBase_LeftHandIndex1',   [ 4.0, 4.0, 3.0 ] ],
+	[ 'RightShoulder_RightArm', [ 0.01, 0.001, 0.001 ] ],
+	[ 'RightArm_RightForeArm',  [ 5.0, 5.0, 1.0 ] ],
+	[ 'RightForeArm_RightHand', [ 5.0, 5.0, 1.0 ] ],
+	[ 'RightFingerBase_RightHandIndex1', [ 4.0, 4.0, 3.0 ] ],
+]}" />
 <!-- ######################################## -->
 <xacro:macro name="make_one_human_collision_model" params="id sW:=^|0.44
@@ -38,8 +60,41 @@
 	</xacro:if>
 </xacro:macro>
+<!-- ############################################################ -->
+<xacro:macro name="make_one_scaling" params="bone sX sY sZ suffix:='_collision'
+		szPoseAttr:=''">
+	<xacro:property name="_bNoPose" value="${szPoseAttr == ''}" />
+	<xacro:unless value="${_bNoPose}">
+	<scaling collision="${bone}${suffix}" scale="${sX} ${sY} ${sZ}"
+		pose="${szPoseAttr}" />
+	</xacro:unless>
+	<xacro:if value="${_bNoPose}">
+	<scaling collision="${bone}${suffix}" scale="${sX} ${sY} ${sZ}" />
+	</xacro:if>
+</xacro:macro>
 <!-- ######################################## -->
+<xacro:macro name="loop_through_scaling" params="scaling_list:=^">
+	<xacro:if value="${scaling_list}">
+		<xacro:property name="_cfg_scale" value="${list( scaling_list.pop(0))}"
+			/>
+		<xacro:property name="RET" value="${_cfg_scale.append( '')}" />
+		<xacro:induce_eval />
+		<xacro:make_one_scaling bone="${_cfg_scale[0]}"
+			sX="${_cfg_scale[1][0]}"
+			sY="${_cfg_scale[1][1]}"
+			sZ="${_cfg_scale[1][2]}"
+			szPoseAttr="${_cfg_scale[2]}" />
+		<xacro:loop_through_scaling />
+	</xacro:if>
+</xacro:macro>
+<!-- ############################################################ -->
 <xacro:macro name="make_one_actor_traj_model" params="id pX pY vel colour
 		pTrajXY anim:='walking' pZ:=1.0 oX:='__PI_HALF' oY:=-0.0 oZ:='__PI'
-		obs_margin:=0.2 rname:='servicebot'">
+		obs_margin:=0.2 rname:='servicebot' bScaleSkel4Collision:=False">
+	<xacro:property name="_trajActorPluginFile"
+		value="libTrajectoryActorPlugin.so" />
+	<xacro:if value="${bScaleSkel4Collision}">
+		<xacro:property name="_trajActorPluginFile"
+			value="libTrajectoryActorExtendedPlugin.so" />
+	</xacro:if>
 <actor name="human_${id}">
 	<!-- Starting pose, nice for when the world is reset -->
@@ -55,10 +110,16 @@
 	<xacro:property name="_vel" value="${pRet.pop()}" />
 	<xacro:induce_eval RET="${_vel}" />
-	<plugin name="trajectory" filename="libTrajectoryActorPlugin.so">
+	<plugin name="trajectory" filename="${_trajActorPluginFile}">
 		<xacro:make_pose_seq pPoseXY="${list( pTrajXY)}" />
 		<velocity>${_vel[1:]}</velocity>
 		<obstacle_margin>${obs_margin}</obstacle_margin>
 		<obstacle>${rname}</obstacle>
+		<debug on_load="False" on_update="False" />
+		<xacro:if value="${bScaleSkel4Collision}">
+		<xacro:loop_through_scaling
+			scaling_list="${list( actor_bone_scaling_map)}" />
+		</xacro:if>
 	</plugin>
+	<xacro:unless value="${bScaleSkel4Collision}">
 	<!-- Enable collisions -->
 	<plugin name="attach_model" filename="libAttachModelPlugin.so">
@@ -70,4 +131,5 @@
 		</link>
 	</plugin>
+	</xacro:unless>
 </actor>
 </xacro:macro>
