Commit message: Defined new <xacro:macro> "loop_through_custom_cfg_to_map", as a future replacement for "loop_through_custom_cfg", whereby the former will loop recursively to parse a sequence of command-line custom configuration options into a return dictionary variable, as opposed to directly generating the corresponding block of custom .sdf mark-up within its own body (for the latter). This will make for cleaner future extension of customised SDF mark-up blocks.
<xacro:macro> "loop_through_custom_cfg": BUG FIX - added str() cast on each custom configuration value being tested so as to support truncated values that contain only digits (which will be stored as numbers within xacro parser).
Also extended functionality of macro so that alternative customisation configuration values to those for setting actor trajectories can be introduced that do not involve specification of trajectory lists.

File: worlds/lib_custom.world.xacro (robot description, xacro)
@@ -1,4 +1,36 @@
 <?xml version="1.0" ?>
 <robot xmlns:xacro="http://www.ros.org/wiki/xacro">
+<!-- ######################################## -->
+<xacro:macro name="loop_through_custom_cfg_to_map" params="pRetMap:=^
+		custom_list:=^ _bDebug:=^|False">
+	<xacro:if value="${custom_list}">
+		<xacro:property name="_cfg_opt" value="${custom_list.pop(0)}" />
+		<xacro:property name="_val" value="None" />
+		<xacro:property name="_sepIdx" value="${str(_cfg_opt).find( '.')}" />
+		<xacro:property name="_key" value="${str(_cfg_opt)[:_sepIdx]}" />
+		<xacro:if value="${_sepIdx != -1}">
+			<xacro:property name="_val" value="${str(_cfg_opt)[_sepIdx+1:]}" />
+		</xacro:if>
+		<xacro:unless value="${_sepIdx != -1}">
+			<xacro:property name="_key" value="${str(_cfg_opt)}" />
+		</xacro:unless>
+		<xacro:property name="_bRepeated" value="${ _key in pRetMap}" />
+		<xacro:if value="${_bRepeated}">
+			<error>key [${_key}] already exists with value (${pRetMap.get(
+				_key)})</error>
+		</xacro:if>
+		<xacro:if value="${_bDebug}">
+		<_cfg_opt>${_cfg_opt}</_cfg_opt>
+		<_cfg_key>${_key}</_cfg_key>
+		<_cfg_val>${_val}</_cfg_val>
+		</xacro:if>
+		<xacro:unless value="${_bRepeated}">
+			<xacro:property name="_tmp"
+				value="${pRetMap.setdefault( _key, _val)}" />
+			<xacro:induce_eval RET="${_tmp}" />
+		</xacro:unless>
+		<xacro:loop_through_custom_cfg_to_map />
+	</xacro:if>
+</xacro:macro>
 <!-- ######################################## -->
 <xacro:macro name="loop_through_custom_cfg" params="rname:=^ custom_list:=^
@@ -11,11 +43,11 @@
 		<xacro:property name="_shirt" value="" />
 		<xacro:property name="_traj" value="${[]}" />
-		<xacro:if value="${_cfg_opt.endswith( '.a')}">
+		<xacro:if value="${str(_cfg_opt).endswith( '.a')}">
 			<xacro:property name="_vel" value="0.9" />
 		</xacro:if>
-		<xacro:if value="${_cfg_opt.endswith( '.b')}">
+		<xacro:if value="${str(_cfg_opt).endswith( '.b')}">
 			<xacro:property name="_vel" value="1.05" />
 		</xacro:if>
-		<xacro:if value="${_cfg_opt.endswith( '.c')}">
+		<xacro:if value="${str(_cfg_opt).endswith( '.c')}">
 			<xacro:property name="_vel" value="1.2" />
 		</xacro:if>
@@ -83,4 +115,5 @@
 			]}" />
 		</xacro:if>
+		<xacro:if value="${_traj}">
 		<xacro:make_one_human_collision_model id="${_human}" />
 		<xacro:make_one_actor_traj_model id="${_human}" pX="${_traj[0][0]}"
@@ -93,4 +126,5 @@
 		<_traj>${_traj}</_traj>
 		</xacro:if>
+		</xacro:if>
 		<xacro:loop_through_custom_cfg />
 	</xacro:if>
