Commit message: eval_to_bool - new marco to generalise convoluted logic needed for parsing boolean command-line argument values from a raw-valued xacro:arg into a xacro:property. Added new xacro:arg optional command-line arguments "have_gpu" & "rev_joint_velodyne" to respectively support dynamic switching between: gpu & non-gpu plugins (for Hokuyo & apparently also for Velodyne); and between Velodyne sensor that incorporates a revolute joint (for full spherical scans) versus a simpler design without a joint (for half-spherical scan).

File: worlds/service.world.xacro (robot description, xacro)
@@ -9,9 +9,39 @@
 <xacro:include filename="../plugins/camera.xacro" />
 <xacro:include filename="../plugins/kinect.xacro" />
+<xacro:include filename="../plugins/hokuyo.xacro" />
+<xacro:include filename="../plugins/velodyne.xacro" />
+<!-- ######################################## -->
+<xacro:macro name="eval_to_bool" params="val pRet:=^ _bDebug:=False">
+	<xacro:property name="RET" value="" />
+	<xacro:property name="_bRet" value="${False}" />
+	<xacro:property name="_val" value="${str( val).strip().lower()}" />
+	<xacro:if value="${(_val != '') and (
+			(_val == 'true') or (_val == 'yes') or (_val == 'on') or
+			(str(_val).isdigit() and (int(_val) != 0)) )}">
+		<xacro:property name="_bRet" value="${True}" />
+	</xacro:if>
+	<xacro:property name="RET" value="${pRet.append( _bRet)}" />
+	<xacro:induce_eval />
+	<xacro:if value="${_bDebug}">
+		<eval_2_bool>val=${val} => ${_bRet}</eval_2_bool>
+	</xacro:if>
+</xacro:macro>
+<!-- ######################################## -->
 <xacro:arg name="robot_name" default="servicebot" />
 <xacro:arg name="custom_cfg" default="1.a" />
+<xacro:arg name="have_gpu" default="True" />
+<xacro:arg name="rev_joint_velodyne" default="False" />
 <xacro:property name="_custom_cfg" value="$(arg custom_cfg)" />
 <xacro:property name="no_custom" value="${str(_custom_cfg).strip() == '0'}"
 	/>
+<xacro:property name="_gpu_arg" value="$(arg have_gpu)" />
+<xacro:property name="_have_gpu" value="${str( _gpu_arg).strip().lower()}" />
+<xacro:property name="use_gpu" value="${(_have_gpu != '') and (
+		(_have_gpu == 'true') or (_have_gpu == 'yes') or (_have_gpu == 'on') or
+		(str(_have_gpu).isdigit() and (int(_have_gpu) != 0)) )}"
+	/>
+<xacro:eval_to_bool val="$(arg rev_joint_velodyne)" _bDebug="True" />
+<xacro:property name="revolute_joint_velo" value="${pRet.pop()}" />
+<xacro:induce_eval RET="${revolute_joint_velo}" />
 <xacro:property name="do_public_cafe_default_fixture" value="${no_custom}"
 	/>

Commit message: Added new <xacro:arg> "use_skel_collision" to initialise new global <xacro:property> "use_skeleton_4_collision", for passing to "loop_through_custon_cfg" recursive <xacro:macro> call as its new parameter "bUseSkelCollision".
Added (default disabled) copy of talking actor SDF block (for actor "human_69100") duplicated from example.world of servicesim_competition package, that was use to demonstrate original CollisionActorPlugin Gazebo plugin in the latter, in order to experiment with generating collision links based on .dae-based actor skeleton.

File: worlds/service.world.xacro (robot description, xacro)
@@ -30,4 +30,5 @@
 <xacro:arg name="robot_name" default="servicebot" />
 <xacro:arg name="custom_cfg" default="1.a" />
+<xacro:arg name="use_skel_collision" default="False" />
 <xacro:arg name="have_gpu" default="True" />
 <xacro:arg name="rev_joint_velodyne" default="False" />
@@ -41,5 +42,8 @@
 		(str(_have_gpu).isdigit() and (int(_have_gpu) != 0)) )}"
 	/>
-<xacro:eval_to_bool val="$(arg rev_joint_velodyne)" _bDebug="True" />
+<xacro:eval_to_bool val="$(arg use_skel_collision)" _bDebug="False" />
+<xacro:property name="use_skeleton_4_collision" value="${pRet.pop()}" />
+<xacro:induce_eval RET="${use_skeleton_4_collision}" />
+<xacro:eval_to_bool val="$(arg rev_joint_velodyne)" _bDebug="False" />
 <xacro:property name="revolute_joint_velo" value="${pRet.pop()}" />
 <xacro:induce_eval RET="${revolute_joint_velo}" />
@@ -580,7 +584,146 @@
 	<xacro:property name="_custom_list" value="${_custom_cfg.split(',')}" />
 	<xacro:loop_through_custom_cfg rname="$(arg robot_name)"
+		bUseSkelCollision="${use_skeleton_4_collision}"
 		custom_list="${_custom_list}" />
 </xacro:unless>
 </xacro:unless>
+<xacro:if value="False">
+<actor name="human_69100">
+	<!-- Starting pose, nice for when the world is reset -->
+	<pose>
+		20.5
+		4.0
+		0.0
+		0.0
+		-0.0
+		-3.142
+	</pose>
+	<skin>
+		<filename>model://actor/meshes/SKIN_man_green_shirt.dae</filename>
+	</skin>
+	<animation name="animation">
+		<filename>model://actor/meshes/ANIMATION_talking_b.dae</filename>
+	</animation>
+	<!-- Need one waypoint to idle at -->
+	<script>
+		<trajectory id='0' type='animation'>
+			<waypoint>
+				<time>100</time>
+					<pose>
+						20.5
+						4.0
+						0.0
+						0.0
+						-0.0
+						-3.142
+					</pose>
+			</waypoint>
+		</trajectory>
+	</script>
+	<!-- Enable collisions -->
+<plugin name="actor_collisions_plugin" filename="libCollisionActorPlugin.so">
+  <scaling collision="LHipJoint_LeftUpLeg_collision" scale="
+    0.01
+    0.001
+    0.001
+  "/>
+  <scaling collision="LeftUpLeg_LeftLeg_collision" scale="
+    8.0
+    8.0
+    1.0
+  "/>
+  <scaling collision="LeftLeg_LeftFoot_collision" scale="
+    8.0
+    8.0
+    1.0
+  "/>
+  <scaling collision="LeftFoot_LeftToeBase_collision" scale="
+    4.0
+    4.0
+    1.5
+  "/>
+  <scaling collision="RHipJoint_RightUpLeg_collision" scale="
+    0.01
+    0.001
+    0.001
+  "/>
+  <scaling collision="RightUpLeg_RightLeg_collision" scale="
+    8.0
+    8.0
+    1.0
+  "/>
+  <scaling collision="RightLeg_RightFoot_collision" scale="
+    8.0
+    8.0
+    1.0
+  "/>
+  <scaling collision="RightFoot_RightToeBase_collision" scale="
+    4.0
+    4.0
+    1.5
+  "/>
+  <scaling collision="LowerBack_Spine_collision" scale="
+    12.0
+    20.0
+    5.0
+  " pose="0.05 0 0 0 -0.2 0"/>
+  <scaling collision="Spine_Spine1_collision" scale="
+    0.01
+    0.001
+    0.001
+  "/>
+  <scaling collision="Neck_Neck1_collision" scale="
+    0.01
+    0.001
+    0.001
+  "/>
+  <scaling collision="Neck1_Head_collision" scale="
+    5.0
+    5.0
+    3.0
+  "/>
+  <scaling collision="LeftShoulder_LeftArm_collision" scale="
+    0.01
+    0.001
+    0.001
+  "/>
+  <scaling collision="LeftArm_LeftForeArm_collision" scale="
+    5.0
+    5.0
+    1.0
+  "/>
+  <scaling collision="LeftForeArm_LeftHand_collision" scale="
+    5.0
+    5.0
+    1.0
+  "/>
+  <scaling collision="LeftFingerBase_LeftHandIndex1_collision" scale="
+    4.0
+    4.0
+    3.0
+  "/>
+  <scaling collision="RightShoulder_RightArm_collision" scale="
+    0.01
+    0.001
+    0.001
+  "/>
+  <scaling collision="RightArm_RightForeArm_collision" scale="
+    5.0
+    5.0
+    1.0
+  "/>
+  <scaling collision="RightForeArm_RightHand_collision" scale="
+    5.0
+    5.0
+    1.0
+  "/>
+  <scaling collision="RightFingerBase_RightHandIndex1_collision" scale="
+    4.0
+    4.0
+    3.0
+  "/>
+</plugin>
+</actor>
+</xacro:if>
 	<!-- Idling actors -->
 <xacro:if value="${do_actor_default_idle}">

Commit message: Added new utility <xacro:macro> "ensure_path_suffix", that will process input parameter string value to ensure that it is terminated with path separator (i.e. "/") if it is non-trivial. Added new <xacro:arg>s "vis_lidar_2d" & "vis_lidar_3d" to respectively initialise new global <xacro:property>s "visible_lidar_2d" & "visible_lidar_3d", for passing respectively to "plugin_sensor_hokuyo" & "plugin_sensor_velodyne" <xacro:macro> calls, so that toggling of visualisation of 2D & 3D lidar rays in Gazebo can be controlled from command line.

File: worlds/service.world.xacro (robot description, xacro)
@@ -28,4 +28,18 @@
 </xacro:macro>
 <!-- ######################################## -->
+<xacro:macro name="ensure_path_suffix" params="val pRet:=^ _bDebug:=False">
+	<xacro:property name="RET" value="" />
+	<xacro:property name="_ret" value="${val}" />
+	<xacro:property name="_val" value="${str( val).strip().lower()}" />
+	<xacro:if value="${(_val != '') and (_val[-1] != '/')}">
+		<xacro:property name="_ret" value="${_val}/" />
+	</xacro:if>
+	<xacro:property name="RET" value="${pRet.append( _ret)}" />
+	<xacro:induce_eval />
+	<xacro:if value="${_bDebug}">
+		<ensure_path_suffix>val=${val} => ${_val}</ensure_path_suffix>
+	</xacro:if>
+</xacro:macro>
+<!-- ######################################## -->
 <xacro:arg name="robot_name" default="servicebot" />
 <xacro:arg name="custom_cfg" default="1.a" />
@@ -33,4 +47,6 @@
 <xacro:arg name="have_gpu" default="True" />
 <xacro:arg name="rev_joint_velodyne" default="False" />
+<xacro:arg name="vis_lidar_2d" default="False" />
+<xacro:arg name="vis_lidar_3d" default="False" />
 <xacro:property name="_custom_cfg" value="$(arg custom_cfg)" />
 <xacro:property name="no_custom" value="${str(_custom_cfg).strip() == '0'}"
@@ -48,4 +64,10 @@
 <xacro:property name="revolute_joint_velo" value="${pRet.pop()}" />
 <xacro:induce_eval RET="${revolute_joint_velo}" />
+<xacro:eval_to_bool val="$(arg vis_lidar_2d)" _bDebug="False" />
+<xacro:property name="visible_lidar_2d" value="${pRet.pop()}" />
+<xacro:induce_eval RET="${visible_lidar_2d}" />
+<xacro:eval_to_bool val="$(arg vis_lidar_3d)" _bDebug="False" />
+<xacro:property name="visible_lidar_3d" value="${pRet.pop()}" />
+<xacro:induce_eval RET="${visible_lidar_3d}" />
 <xacro:property name="do_public_cafe_default_fixture" value="${no_custom}"
 	/>

Commit message: Moved up declaration of <xacro:property> "_custom_list" (used to pass to "loop_through_custom_cfg" macro call) to initialisation block for <xacro:arg> & <xacro:property> globals new top of file. Added call to new <xacro:macro> "loop_through_custom_cfg_to_map" on copy of "_custom_list" list to populate equivalent new global dictionary of custom configuration values, "_pCfgMap". Inserted new optional (on new configuration key in "_pCfgMap") <plugin> block for third-party Gazebo plugin for generating map from Gazebo world, at start of <world> block.

File: worlds/service.world.xacro (robot description, xacro)
@@ -50,6 +50,9 @@
 <xacro:arg name="vis_lidar_3d" default="False" />
 <xacro:property name="_custom_cfg" value="$(arg custom_cfg)" />
-<xacro:property name="no_custom" value="${str(_custom_cfg).strip() == '0'}"
-	/>
+<xacro:property name="no_custom" value="${str(_custom_cfg).strip() == '0'}" />
+<xacro:property name="_custom_list" value="${str(_custom_cfg).split(',')}" />
+<xacro:property name="_pCfgMap" value="${dict()}" />
+<xacro:loop_through_custom_cfg_to_map pRetMap="${_pCfgMap}"
+	custom_list="${list(_custom_list)}" _bDebug="False" />
 <xacro:property name="_gpu_arg" value="$(arg have_gpu)" />
 <xacro:property name="_have_gpu" value="${str( _gpu_arg).strip().lower()}" />
@@ -83,8 +86,27 @@
 <sdf version="1.6">
 <world name="default">
+	<xacro:if value="${(4 in _pCfgMap) or ('x' in _pCfgMap)}">
+	<plugin name='gazebo_occupancy_map' filename='libgazebo_2Dmap_plugin.so'>
+		<!--
+			# map_resolution: in meters, optional, default 0.1
+			# map_z: in meters, optional, default 0.3
+			# map_size_x: in meters, optional, default 10
+			# map_size_y: in meters, optional, default 10
+			# init_robot_x: x coordinate in meters, optional, default 0
+			# init_robot_y: y coordinate in meters, optional, default 0
+		-->
+		<map_resolution>0.1</map_resolution>
+		<map_z>0.76</map_z>
+		<map_size_x>58</map_size_x>
+		<map_size_y>58</map_size_y>
+		<init_robot_x>20.15</init_robot_x>
+		<init_robot_y>1.45</init_robot_y>
+	</plugin>
+	</xacro:if>
 	<debug>
 		<custom_cfg>$(arg custom_cfg)</custom_cfg>
 		<_custom_cfg>${_custom_cfg}</_custom_cfg>
 		<no_custom>${no_custom}</no_custom>
+		<_cfg_map>${str(_pCfgMap)}</_cfg_map>
 		<do_public_cafe_default_fixture>
 			${do_public_cafe_default_fixture}
@@ -604,5 +626,4 @@
 <xacro:unless value="${do_actor_default_dynamic}">
 <xacro:unless value="${no_custom}">
-	<xacro:property name="_custom_list" value="${_custom_cfg.split(',')}" />
 	<xacro:loop_through_custom_cfg rname="$(arg robot_name)"
 		bUseSkelCollision="${use_skeleton_4_collision}"

Commit message: Updated all calls to "include_one_X_db_model" <xacro:macro> for table models to append new optional parameters "bAddCollideBox" & "bVisHack", which are assigned values of global <xacro:property> variables "expand_table_leg" & "hack_collide_vis" respectively, to use extended functionality of "include_one_X_db_model" to add collision box at the same pose as the model.

File: worlds/service.world.xacro (robot description, xacro)
@@ -49,4 +49,6 @@
 <xacro:arg name="vis_lidar_2d" default="False" />
 <xacro:arg name="vis_lidar_3d" default="False" />
+<xacro:arg name="hack_table" default="True" />
+<xacro:arg name="show_hack" default="False" />
 <xacro:property name="_custom_cfg" value="$(arg custom_cfg)" />
 <xacro:property name="no_custom" value="${str(_custom_cfg).strip() == '0'}" />
@@ -73,4 +75,10 @@
 <xacro:property name="visible_lidar_3d" value="${pRet.pop()}" />
 <xacro:induce_eval RET="${visible_lidar_3d}" />
+<xacro:eval_to_bool val="$(arg hack_table)" _bDebug="False" />
+<xacro:property name="expand_table_leg" value="${pRet.pop()}" />
+<xacro:induce_eval RET="${expand_table_leg}" />
+<xacro:eval_to_bool val="$(arg show_hack)" _bDebug="False" />
+<xacro:property name="hack_collide_vis" value="${pRet.pop()}" />
+<xacro:induce_eval RET="${hack_collide_vis}" />
 <xacro:property name="do_public_cafe_default_fixture" value="${no_custom}"
 	/>
