Commit message: Update <xacro:macro> "plugin_sensor_hokuyo" to add call to new utility macro "ensure_path_suffix" to automatically ensure that any non-trivial value of optional parameter "topic_prefix" will be terminated with path separator (i.e. "/").

File: plugins/hokuyo.xacro (robot description, xacro)
@@ -8,4 +8,7 @@
 		M_PI_HALF:='1.5707963267948966' _bDebug:=False
 ">
+	<xacro:ensure_path_suffix val="${topic_prefix}" _bDebug="False" />
+	<xacro:property name="topic_prefix" value="${pRet.pop()}" />
+	<xacro:induce_eval RET="${topic_prefix}" />
 	<xacro:property name="_type" value="ray" />
 	<xacro:property name="_lib" value="libgazebo_ros_laser.so" />
