Commit message: Hived out the 2 main SDF blocks - for control box and end-effector attachment - in separate new .urdf.xacro files (custom_part_control_box.urdf.xacro and custom_part_ee_attachment.urdf.xacro), for better reusability (e.g. to re-use .urdf.xacro for end-effector attachment with stand-alone UR5e [i.e. without mobile base]).

File: urdf/custom.urdf.xacro (robot description, xacro)
@@ -4,58 +4,5 @@
 <robot xmlns:xacro="http://ros.org/wiki/xacro" name="husky">
 -->
-  <xacro:arg name="parent_link_for_custom" default="top_plate_front_link" />
-  <xacro:property name="_parent_link_for_custom"
-      value="$(arg parent_link_for_custom)" />
-  <!-- Control Box Properties -->
-  <xacro:property name="ctrl_box_width" value="0.52" />
-  <xacro:property name="ctrl_box_length" value="0.59" />
-  <xacro:property name="ctrl_box_height" value="0.68" />
-  <link name="control_box" >
-    <visual>
-      <geometry>
-        <box size="${ctrl_box_width} ${ctrl_box_length} ${ctrl_box_height}" />
-      </geometry>
-      <material name="white"/>
-    </visual>
-    <collision>
-      <geometry>
-        <box size="${ctrl_box_width} ${ctrl_box_length} ${ctrl_box_height}" />
-      </geometry>
-    </collision>
-  </link>
-  <joint name="control_box_mount_joint" type="fixed">
-    <parent link="${_parent_link_for_custom}" />
-    <child link="control_box" />
-<!--
-    <axis xyz="0 0 1"/>
--->
-    <origin xyz="-${ctrl_box_width} 0 ${ctrl_box_height/2.0}" rpy="0 0 0" />
-  </joint>
-  <!-- End-effector attachment -->
-  <xacro:property name="_robot_arm_link_prefix" value="ur_arm_" />
-  <xacro:property name="_extra_mesh_pkg_path"
-      value="package://mobile_manipulator_moveit_config/meshes/ur5e/" />
-  <link name="EEF" >
-    <visual>
-      <origin rpy="0 ${_M_PI} ${_M_PI}" xyz="0.26 0.0 0.0"/>
-      <geometry>
-        <mesh filename="${_extra_mesh_pkg_path}visual/circle_tray.STL" />
-      </geometry>
-      <material name="LightGrey">
-        <color rgba="0.7 0.7 0.7 1.0"/>
-      </material>
-    </visual>
-    <collision>
-      <origin rpy="0 3.14159 3.14159" xyz="0.26 0.0 0.0"/>
-      <geometry>
-        <mesh filename="${_extra_mesh_pkg_path}visual/circle_tray.STL" />
-      </geometry>
-    </collision>
-  </link>
-  <joint name="EEF_mount_joint" type="fixed">
-    <parent link="${_robot_arm_link_prefix}ee_link"/>
-    <child link="EEF"/>
-    <axis xyz="0 0 1"/>
-    <origin rpy="0 0 0" xyz="0 0 0"/>
-  </joint>
+  <xacro:include filename="custom_part_control_box.urdf.xacro" />
+  <xacro:include filename="custom_part_ee_attachment.urdf.xacro" />
 </robot>

Commit message: Updated to <xacro:include> new .urdf.xacro files: custom_part_sensor_kinect; custom_part_ee_gripper; custom_part_world_frame. Inclusion of custom_part_ee_gripper.urdf.xacro is made mutually exclusive with existing custom_part_ee_attachment.urdf.xacro depending on value of new externally-set <xacro:arg> "ee_type". Inclusion of custom_part_world_frame.urdf.xacro is made conditional of new externally-set <xacro:arg> "add_world_link".

File: urdf/custom.urdf.xacro (robot description, xacro)
@@ -4,5 +4,19 @@
 <robot xmlns:xacro="http://ros.org/wiki/xacro" name="husky">
 -->
+  <xacro:include filename="lib_util.urdf.xacro" />
   <xacro:include filename="custom_part_control_box.urdf.xacro" />
-  <xacro:include filename="custom_part_ee_attachment.urdf.xacro" />
+  <xacro:include filename="custom_part_sensor_kinect.urdf.xacro" />
+  <xacro:property name="_ee_type" value="$(arg ee_type)" />
+  <xacro:if value="${_ee_type == 'tray'}">
+    <xacro:include filename="custom_part_ee_attachment.urdf.xacro" />
+  </xacro:if>
+  <xacro:if value="${_ee_type == 'hand'}">
+    <xacro:include filename="custom_part_ee_gripper.urdf.xacro" />
+  </xacro:if>
+  <xacro:eval_to_bool val="$(arg add_world_link)" _bDebug="False" />
+  <xacro:property name="_bAddWorldLink" value="${pRet.pop()}" />
+  <xacro:induce_eval RET="${_bAddWorldLink}" />
+  <xacro:if value="${_bAddWorldLink}">
+    <xacro:include filename="custom_part_world_frame.urdf.xacro" />
+  </xacro:if>
 </robot>
