Commit message: Extended functionality of "add_virtual_joint" <xacro:macro> by adding new "pos_limit_abs" optional param, such that: if "pos_limit_abs" has a valid float value, then the <limit> declaration will use explicit values of negative and positive ${pos_limit_abs} for "lower" & "upper" attribute values respectively; or otherwise, leave the "lower" & "upper" <limit> attribute values unspecified (i.e. no limits to <joint>).

File: urdf/transmission.urdf.xacro (robot description, xacro)
@@ -69,5 +69,11 @@
 <!-- ######################################## -->
 <xacro:macro name="add_virtual_joint" params="name type parent child axis
-		base_link_z_offset:=0.0 effort_limit:=1000.0 vel_limit:=0.5">
+		base_link_z_offset:=0.0 effort_limit:=1000.0 vel_limit:=0.5
+		pos_limit_abs:=50.0">
+	<xacro:property name="_bNoLimit" value="${True}" />
+	<xacro:if value="${str(pos_limit_abs).replace('.','',1).isdigit() and
+			(float(pos_limit_abs) != 0.0)}">
+		<xacro:property name="_bNoLimit" value="${False}" />
+	</xacro:if>
 	<xacro:property name="_x" value="${(0,1)[ axis == 'x']}" />
 	<xacro:property name="_y" value="${(0,1)[ axis == 'y']}" />
@@ -76,6 +82,11 @@
 		<parent link="${parent}" />
 		<child link="${child}" />
-		<limit effort="${effort_limit}" lower="-5" upper="5"
-			velocity="${vel_limit}" />
+		<xacro:if value="${_bNoLimit}">
+			<limit effort="${effort_limit}" velocity="${vel_limit}" />
+		</xacro:if>
+		<xacro:unless value="${_bNoLimit}">
+			<limit effort="${effort_limit}" velocity="${vel_limit}"
+				lower="-${pos_limit_abs}" upper="${pos_limit_abs}" />
+		</xacro:unless>
 		<axis xyz="${_x} ${_y} ${_z}" />
 		<origin xyz="0 0 ${base_link_z_offset}" />
@@ -89,4 +100,5 @@
 		_bDebug:=False">
 	<xacro:property name="_szAxisPrefix" value="" />
+	<xacro:property name="_fPosLimitAbs" value="50.0" />
 	<xacro:if value="${szJointType == 'prismatic'}">
 		<xacro:property name="_szAxisPrefix" value="t" />
@@ -94,4 +106,5 @@
 	<xacro:if value="${szJointType == 'revolute'}">
 		<xacro:property name="_szAxisPrefix" value="r" />
+		<xacro:property name="_fPosLimitAbs" value="${pi}" />
 	</xacro:if>
 	<xacro:property name="_szJ" value="${szJ.strip()}" />
@@ -110,5 +123,6 @@
 		type="${szJointType}" parent="${szParent}" child="${_szL}"
 		axis="${axis}" base_link_z_offset="${base_link_z_offset}"
-		effort_limit="${effort_limit}" vel_limit="${vel_limit}" />
+		effort_limit="${effort_limit}" vel_limit="${vel_limit}"
+		pos_limit_abs="${_fPosLimitAbs}" />
 	<xacro:add_transmission szJ="${_szJ}"
 		szJointPrefix="${szJointVirtualPrefix}" _bDebug="${_bDebug}" />

Commit message: Revised "default_inertial" <macro> to change hard-coded values for <inertia> "ixx", "iyy" & "izz" attribute values from 1.0 to new i_axis_default parameter with default value. Note: default value should be revised from 1.0 to something small (e.g. 0.0001) in future so that virtual links connecting a robot base to a world link will not have too much inertia (check by enabling inertia view in Gazebo).

File: urdf/transmission.urdf.xacro (robot description, xacro)
@@ -45,12 +45,12 @@
 <!-- ######################################## -->
 <!-- ######################################## -->
-<xacro:macro name="default_inertial" params="mass:=1.0">
+<xacro:macro name="default_inertial" params="mass:=1.0 i_axis_default:=1.0000">
 	<inertial>
 		<mass value="${mass}" />
 		<origin xyz="0 0 0" rpy="0 0 0" />
 		<inertia
-			ixx="1.0" ixy="0.0" ixz="0.0"
-			iyy="1.0" iyz="0.0"
-			izz="1.0" />
+			ixx="${i_axis_default}" ixy="0.0" ixz="0.0"
+			iyy="${i_axis_default}" iyz="0.0"
+			izz="${i_axis_default}" />
 	</inertial>
 </xacro:macro>
