Commit message: Commented out <material> declaration for "aluminum" (otherwise will get duplicate material declaration) and replaced it with <material> declaration using hard-coded <color> element.

File: urdf/_d435-copied_from_realsense2_description.urdf.xacro (robot description, xacro)
@@ -63,5 +63,10 @@
             <box size="${d435_cam_depth} ${d435_cam_width} ${d435_cam_height}"/>
           </geometry>
+          <material>
+            <color rgba="0.5 0.5 0.5 1"/>
+          </material>
+<!--
           <material name="aluminum"/>
+-->
         </xacro:unless>
       </visual>
