Commit message: Updated to check current ROS_DISTRO environment variable and if it is "noetic", to <include> local customised copy of _d435.urdf.xacro from realsense2_description package, and to call different macro (originally "intel_realsense_mount" on Kinetic) named "realsense_sensor" with different param name list. This revision is to cater for most recent upgrade to ros-noetic-husky-description package, in which the morons maintaining it have completely broken the package by renaming the macro from "intel_realsense_mount" to "realsense_sensor". In addition, the new intel_realsense.urdf.xacro includes different versions of realsense models' URDF, all of which are broken because they all redeclare <material> for "aluminum", which causes an error in xacro during loading.

File: urdf/custom_part_sensor_kinect.urdf.xacro (robot description, xacro)
@@ -5,4 +5,13 @@
   <xacro:property name="_parent_link_for_sensor"
       value="$(arg parent_link_for_sensor)" />
+  <xacro:property name="_ros_distro" value="$(optenv ROS_DISTRO)" />
+  <xacro:property name="_is_kinetic" value="${_ros_distro == 'kinetic'}" />
+  <xacro:unless value="${_is_kinetic}">
+    <xacro:include filename="_d435.urdf.xacro" />
+<!--
+    <xacro:include
+      filename="$(find realsense2_description)/urdf/_d435.urdf.xacro" />
+-->
+  </xacro:unless>
   <!-- Control Box Properties -->
   <xacro:property name="ctrl_box_width" value="0.52" />
@@ -17,6 +26,14 @@
       <child link="realsense_mount_front" />
     </joint>
-    <xacro:intel_realsense_mount prefix="camera1" topic="realsense_front"
-      parent_link="realsense_mount_front"/>
+    <xacro:if value="${_is_kinetic}">
+      <xacro:intel_realsense_mount prefix="camera1" topic="realsense_front"
+        parent_link="realsense_mount_front"/>
+    </xacro:if>
+    <xacro:unless value="${_is_kinetic}">
+      <xacro:realsense_sensor prefix="camera1" topic="realsense_front"
+          parent="realsense_mount_front" include="0">
+        <origin xyz="0.0115 0 0.0100" rpy="0 0 0" />
+      </xacro:realsense_sensor>
+    </xacro:unless>
   </xacro:if>
   <xacro:if value="${True}">
@@ -28,6 +45,14 @@
       <child link="realsense_mount_right" />
     </joint>
-    <xacro:intel_realsense_mount prefix="camera2" topic="realsense_right"
-      parent_link="realsense_mount_right"/>
+    <xacro:if value="${_is_kinetic}">
+      <xacro:intel_realsense_mount prefix="camera2" topic="realsense_right"
+        parent_link="realsense_mount_right"/>
+    </xacro:if>
+    <xacro:unless value="${_is_kinetic}">
+      <xacro:realsense_sensor prefix="camera2" topic="realsense_right"
+          parent="realsense_mount_right" include="0">
+        <origin xyz="0.0115 0 0.0100" rpy="0 0 0" />
+      </xacro:realsense_sensor>
+    </xacro:unless>
   </xacro:if>
 </robot>

Commit message: Additional comments to: document change in top-level macro name of official Husky (i.e Clearpath Robotics) implementation of Realsense camera URDF; explain need to making local copy of official ros-kinetic-realsense2-description package's _d435.urdf.xacro file (to comment out <include> of material file containing <material> elements that leads to xacro is complaining of <material> redefinition).

File: urdf/custom_part_sensor_kinect.urdf.xacro (robot description, xacro)
@@ -5,7 +5,18 @@
   <xacro:property name="_parent_link_for_sensor"
       value="$(arg parent_link_for_sensor)" />
+  <!--
+    # Name of top-level macro for Realsense camera has been changed after ROS
+    # Kinetic: from "intel_realsense_mount" to "realsense_sensor"; and with
+    # different parameter names.
+  -->
   <xacro:property name="_ros_distro" value="$(optenv ROS_DISTRO)" />
   <xacro:property name="_is_kinetic" value="${_ros_distro == 'kinetic'}" />
   <xacro:unless value="${_is_kinetic}">
+    <!--
+      # NOTE: local copy made of original urdf/_d435.urdf.xacro in
+      # realsense2_description package in order to patch original,
+      # by commenting out <xacro:include> of material file which leads to
+      # xacro complaining about some <material> being redefined.
+    -->
     <xacro:include filename="_d435.urdf.xacro" />
 <!--

Commit message: Updated logic to add check for ROS_VERSION, so that condition for deciding to call <xacro:intel_realsense_mount> v.s. <xacro:realsense_sensor> macros works for ROS2 (Humble) as well.

File: urdf/custom_part_sensor_kinect.urdf.xacro (robot description, xacro)
@@ -10,6 +10,9 @@
     # different parameter names.
   -->
+  <xacro:property name="_ros_version" value="$(optenv ROS_VERSION 1)" />
   <xacro:property name="_ros_distro" value="$(optenv ROS_DISTRO)" />
   <xacro:property name="_is_kinetic" value="${_ros_distro == 'kinetic'}" />
+  <xacro:property name="_is_kinetic_or_ros2"
+    value="${_is_kinetic or (_ros_version == 2)}" />
   <xacro:unless value="${_is_kinetic}">
     <!--
@@ -30,4 +33,7 @@
   <xacro:property name="ctrl_box_height" value="0.68" />
   <xacro:if value="${True}">
+    <!--
+      # Front-side mounted/facing camera.
+    -->
     <link name="realsense_mount_front"/>
     <joint name="realsense_mount_front_joint" type="fixed">
@@ -37,9 +43,9 @@
       <child link="realsense_mount_front" />
     </joint>
-    <xacro:if value="${_is_kinetic}">
+    <xacro:if value="${_is_kinetic_or_ros2}">
       <xacro:intel_realsense_mount prefix="camera1" topic="realsense_front"
         parent_link="realsense_mount_front"/>
     </xacro:if>
-    <xacro:unless value="${_is_kinetic}">
+    <xacro:unless value="${_is_kinetic_or_ros2}">
       <xacro:realsense_sensor prefix="camera1" topic="realsense_front"
           parent="realsense_mount_front" include="0">
@@ -49,4 +55,7 @@
   </xacro:if>
   <xacro:if value="${True}">
+    <!--
+      # Right-side mounted/facing camera.
+    -->
     <link name="realsense_mount_right"/>
     <joint name="realsense_mount_right_joint" type="fixed">
@@ -56,9 +65,9 @@
       <child link="realsense_mount_right" />
     </joint>
-    <xacro:if value="${_is_kinetic}">
+    <xacro:if value="${_is_kinetic_or_ros2}">
       <xacro:intel_realsense_mount prefix="camera2" topic="realsense_right"
         parent_link="realsense_mount_right"/>
     </xacro:if>
-    <xacro:unless value="${_is_kinetic}">
+    <xacro:unless value="${_is_kinetic_or_ros2}">
       <xacro:realsense_sensor prefix="camera2" topic="realsense_right"
           parent="realsense_mount_right" include="0">
