Commit message: Replaced hard-coded "ur_arm_" values in: <xacro:property> value declaration for "_robot_arm_link_prefix" with reference to externally declared $(arg robot_arm_link_prefix); and, "prefix" parameter to <xacro:ur5e_robot> macro call with reference to ${_robot_arm_link_prefix}.

File: urdf/husky_ur5_e_description.urdf.xacro (robot description, xacro)
@@ -8,5 +8,6 @@
       value="$(arg parent_link_for_arm)" />
   <xacro:include filename="$(find ur_e_description)/urdf/ur5e.urdf.xacro" />
-  <xacro:property name="_robot_arm_link_prefix" value="ur_arm_" />
+  <xacro:property name="_robot_arm_link_prefix"
+      value="$(arg robot_arm_link_prefix)" />
   <joint name="arm_mount_joint" type="fixed">
     <parent link="${_parent_link_for_arm}" />
@@ -15,4 +16,4 @@
         rpy="$(optenv HUSKY_UR_RPY 0 0 0)" />
   </joint>
-  <xacro:ur5e_robot prefix="ur_arm_" joint_limited="true" />
+  <xacro:ur5e_robot prefix="${_robot_arm_link_prefix}" joint_limited="true" />
 </robot>

Commit message: Added check for ROS_VERSION and logic to set correct base-name of UR link for mounting end-effector, and <include> different top-level xacro macro file (ur5e.urdf.xacro v.s. ur_macro.xacro) for both ROS(1) Kinetic and ROS2 Humble. Bracketed call to <xacro:ur5e> macro within test condition for ROS_VERSION == 1, and added new conditional block (on ROS_VERSION == 2) for calling <xacro:ur_robot> macro for ROS2 (Humble), including presetting a few default <arg> values for passing as params into <xacro:ur_robot>. Bracketed declaration of <joint> "arm_mount_joint" to only be applicable for ROS_VERSION == 1, as <xacro:ur_robot> macro for ROS2 (Humble) specifies its own joint for mounting end-effector.

File: urdf/husky_ur5_e_description.urdf.xacro (robot description, xacro)
@@ -7,7 +7,26 @@
   <xacro:property name="_parent_link_for_arm"
       value="$(arg parent_link_for_arm)" />
-  <xacro:include filename="$(find ur_e_description)/urdf/ur5e.urdf.xacro" />
   <xacro:property name="_robot_arm_link_prefix"
       value="$(arg robot_arm_link_prefix)" />
+  <xacro:property name="_ros_version" value="$(optenv ROS_VERSION 1)" />
+  <xacro:if value="${_ros_version == 1}">
+    <xacro:arg name="robot_arm_ee_attach_link_base_name" default="ee_link" />
+  </xacro:if>
+  <xacro:if value="${_ros_version == 2}">
+    <xacro:arg name="robot_arm_ee_attach_link_base_name" default="flange" />
+  </xacro:if>
+<!--
+  <DEBUG>ROS_VERSION=${_ros_version}</DEBUG>
+-->
+  <xacro:if value="${_ros_version == 1}">
+    <xacro:include filename="$(find ur_e_description)/urdf/ur5e.urdf.xacro" />
+  </xacro:if>
+  <xacro:if value="${_ros_version == 2}">
+<!--
+    <DEBUG>find(ur_description)=$(find ur_description)</DEBUG>
+-->
+    <xacro:include filename="$(find ur_description)/urdf/ur_macro.xacro" />
+  </xacro:if>
+  <xacro:if value="${_ros_version == 1}">
   <joint name="arm_mount_joint" type="fixed">
     <parent link="${_parent_link_for_arm}" />
@@ -16,4 +35,41 @@
         rpy="$(optenv HUSKY_UR_RPY 0 0 0)" />
   </joint>
-  <xacro:ur5e_robot prefix="${_robot_arm_link_prefix}" joint_limited="true" />
+  </xacro:if>
+  <xacro:if value="${_ros_version == 1}">
+    <xacro:ur5e_robot prefix="${_robot_arm_link_prefix}" joint_limited="true" />
+  </xacro:if>
+  <xacro:if value="${_ros_version == 2}">
+    <xacro:arg name="ur_type" default="ur5e" />
+    <xacro:property name="_ur_type_config_path"
+      value="$(find ur_description)/config/$(arg ur_type)" />
+    <xacro:arg name="joint_limit_params"
+      default="${_ur_type_config_path}/joint_limits.yaml"/>
+    <xacro:arg name="kinematics_params"
+      default="${_ur_type_config_path}/default_kinematics.yaml"/>
+    <xacro:arg name="physical_params"
+      default="${_ur_type_config_path}/physical_parameters.yaml"/>
+    <xacro:arg name="visual_params"
+      default="${_ur_type_config_path}/visual_parameters.yaml"/>
+    <xacro:property name="initial_positions_file"
+      value="$(find ur_description)/config/initial_positions.yaml" />
+    <xacro:ur_robot
+      name="$(arg ur_type)"
+      tf_prefix="${_robot_arm_link_prefix}"
+      parent="${_parent_link_for_arm}"
+      joint_limits_parameters_file="$(arg joint_limit_params)"
+      kinematics_parameters_file="$(arg kinematics_params)"
+      physical_parameters_file="$(arg physical_params)"
+      visual_parameters_file="$(arg visual_params)"
+      transmission_hw_interface=""
+      sim_gazebo="true"
+      sim_ignition="false"
+      initial_positions="${xacro.load_yaml(initial_positions_file)}"
+      script_filename=""
+      output_recipe_filename=""
+      input_recipe_filename=""
+    >
+      <origin xyz="$(optenv HUSKY_UR_XYZ -0.18 0.0 ${ctrl_box_height/2.0})"
+        rpy="$(optenv HUSKY_UR_RPY 0 0 0)" />
+    </xacro:ur_robot>
+  </xacro:if>
 </robot>
