Commit message: Replicated global <xacro:property> "ctrl_box_height" that is referenced from within husky_ur5_e_description.urdf.xacro, from within custom.urdf.xacro into this xacro, as husky_ur5_e_description.urdf.xacro needs to be include ahead of custom.urdf.xacro so that MoveIt Setup Assistant does not complain about parent links (in custom.urdf.xacro) not being defined, but at the same time ensure that "ctrl_box_height" property referenced within husky_ur5_e_description.urdf.xacro is set.

File: urdf/husky_ur5_e_for_wp2.urdf.xacro (robot description, xacro)
@@ -1,6 +1,6 @@
 <?xml version="1.0"?>
+<robot xmlns:xacro="http://ros.org/wiki/xacro" name="husky">
+<!--
 <robot xmlns:xacro="http://ros.org/wiki/xacro">
-<!--
-<robot xmlns:xacro="http://ros.org/wiki/xacro" name="husky">
 -->
   <xacro:arg name="parent_link_for_custom" default="top_plate_front_link" />
@@ -10,5 +10,13 @@
   <xacro:property name="_M_PI" value="${pi}"/>
 -->
+  <!-- Control Box Properties -->
+  <!--
+    # "ctrl_box_height" property replicated here from custom.urdf.xacro so that
+    # husky_ur5_e_description.urdf.xacro can be included ahead of
+    # custom.urdf.xacro, so that stupid setup_assistant won't complain that
+    # parent links referenced in the latter are not defined.
+  -->
+  <xacro:property name="ctrl_box_height" value="0.68" />
+  <xacro:include filename="husky_ur5_e_description.urdf.xacro" />
   <xacro:include filename="custom.urdf.xacro" />
-  <xacro:include filename="husky_ur5_e_description.urdf.xacro" />
 </robot>

Commit message: Added check for ROS_VERSION and logic to set default values of new <arg>s "robot_arm_link_prefix" & "robot_arm_ee_attach_angle_roll", for use within urdf/custom_part_ee_attachment.urdf.xacro (<include>-ed by top-level <include>-ed "custom.urdf.xacro").

File: urdf/husky_ur5_e_for_wp2.urdf.xacro (robot description, xacro)
@@ -24,4 +24,15 @@
   -->
   <xacro:property name="ctrl_box_height" value="0.68" />
+  <xacro:property name="_M_PI" value="${pi}"/>
+  <xacro:property name="_ros_version" value="$(optenv ROS_VERSION 1)" />
+  <xacro:arg name="robot_arm_link_prefix" default="" />
+  <xacro:if value="${_ros_version == 1}">
+    <xacro:property name="_robot_arm_ee_attach_angle_roll" value="0" />
+  </xacro:if>
+  <xacro:if value="${_ros_version == 2}">
+    <xacro:property name="_robot_arm_ee_attach_angle_roll" value="${_M_PI}" />
+  </xacro:if>
+  <xacro:arg name="robot_arm_ee_attach_angle_roll"
+    default="${str( _robot_arm_ee_attach_angle_roll)}" />
   <xacro:include filename="husky_ur5_e_description.urdf.xacro" />
   <xacro:include filename="custom.urdf.xacro" />
