Commit message: Changed hard-coded base-name of "EEF_mount_joint" name ("...ee_link") to new <property> value "_robot_ee_attach_link_base_name" (derived from externally-defined new <arg> "robot_arm_ee_attach_link_base_name" parameter), to cater for change in base-name of UR link for mounting end-effector between official versions of husky_description package URDF from ROS(1) Kinetic to ROS2 Humble. Changed roll value of "EEF_mount_joint" origin from hard-coded value (0) to new <property> value "_roll_attach_angle" (derived from externally-defined new <arg> "robot_arm_ee_attach_angle_roll" parameter, to cater for change in origin orientation of UR link for mounting end-effector between official versions of husky_description package URDF from ROS(1) Kinetic to ROS2 Humble.

File: urdf/custom_part_ee_attachment.urdf.xacro (robot description, xacro)
@@ -4,4 +4,8 @@
   <xacro:property name="_robot_arm_link_prefix"
       value="$(arg robot_arm_link_prefix)" />
+  <xacro:property name="_robot_ee_attach_link_base_name"
+      value="$(arg robot_arm_ee_attach_link_base_name)" />
+  <xacro:property name="_roll_attach_angle"
+      value="$(arg robot_arm_ee_attach_angle_roll)" />
   <!-- End-effector attachment - custom tray -->
   <xacro:property name="_extra_mesh_pkg_path"
@@ -25,8 +29,8 @@
   </link>
   <joint name="EEF_mount_joint" type="fixed">
-    <parent link="${_robot_arm_link_prefix}ee_link"/>
+    <parent link="${_robot_arm_link_prefix}${_robot_ee_attach_link_base_name}"/>
     <child link="EEF"/>
     <axis xyz="0 0 1"/>
-    <origin rpy="0 0 0" xyz="0 0 0"/>
+    <origin rpy="${_roll_attach_angle} 0 0" xyz="0 0 0"/>
   </joint>
 </robot>

Commit message: Added conditional logic to set "_extra_mesh_pkg_path" <property> value to use "file://$(find servicesim_for_wp2)" if ROS_VERSION is 2, instead of "package://servicesim_for_wp2" by default regardless of ROS version.

File: urdf/custom_part_ee_attachment.urdf.xacro (robot description, xacro)
@@ -8,7 +8,14 @@
   <xacro:property name="_roll_attach_angle"
       value="$(arg robot_arm_ee_attach_angle_roll)" />
+  <xacro:property name="_ros_version" value="$(optenv ROS_VERSION 1)" />
   <!-- End-effector attachment - custom tray -->
-  <xacro:property name="_extra_mesh_pkg_path"
-      value="package://servicesim_for_wp2/meshes/end_effector/" />
+  <xacro:if value="${_ros_version == 1}">
+    <xacro:property name="_extra_mesh_pkg_path"
+        value="package://servicesim_for_wp2/meshes/end_effector/" />
+  </xacro:if>
+  <xacro:if value="${_ros_version == 2}">
+    <xacro:property name="_extra_mesh_pkg_path"
+        value="file://$(find servicesim_for_wp2)/meshes/end_effector/" />
+  </xacro:if>
   <link name="EEF" >
     <visual>
