Commit message: Added extra conditional logic to handle ROS2 non-support for "package://" protocol for meshes, and replaced reference(s) to "package://husky_description" with value of new <property> "_mesh_proto_pkg_prefix" which is dynamically initialised to either "package://husky_description" (if ROS_VERSION == 1) or "file://$(find husky_description)" (if ROS_VERSION == 2).

File: urdf/husky_macro-copied_from_humble_husky_description.urdf.xacro (robot description, xacro)
@@ -13,10 +13,30 @@
   <xacro:arg name="is_sim" default="false" />
   <xacro:arg name="urdf_extras" default="$(optenv CPR_URDF_EXTRAS empty.urdf)" />
+    <!-- Hack to get round retarded Gazebo non-support for package://
+         protocol format in ROS2 -->
+    <xacro:property name="_ros_version" value="$(optenv ROS_VERSION 1)" />
+    <xacro:if value="${_ros_version == 1}">
+        <xacro:property name="_default_mesh_proto" value="package" />
+    </xacro:if>
+    <xacro:if value="${_ros_version == 2}">
+        <xacro:property name="_default_mesh_proto" value="file" />
+    </xacro:if>
+    <xacro:arg name="mesh_protocol" default="${_default_mesh_proto}" />
+    <xacro:property name="_mesh_protocol" default="$(arg mesh_protocol)" />
+    <xacro:property name="_mesh_pkg_name" value="husky_description" />
+    <xacro:property name="_default_pkg_loc"
+        value="$(find husky_description)" />
+    <xacro:property name="_mesh_pkg_loc" value="${_mesh_pkg_name}" />
+    <xacro:if value="${_mesh_protocol == 'file'}">
+        <xacro:property name="_mesh_pkg_loc" value="${_default_pkg_loc}" />
+    </xacro:if>
+    <xacro:property name="_mesh_proto_pkg_prefix"
+        value="${_mesh_protocol}://${_mesh_pkg_loc}" />
   <!-- Included URDF/XACRO Files -->
-  <xacro:include filename="$(find husky_description)/urdf/decorations.urdf.xacro" />
-  <xacro:include filename="$(find husky_description)/urdf/wheel.urdf.xacro" />
-  <xacro:include filename="$(find husky_description)/urdf/accessories/intel_realsense.urdf.xacro"/>
-  <xacro:include filename="$(find husky_description)/urdf/accessories/sick_lms1xx_mount.urdf.xacro"/>
-  <xacro:include filename="$(find husky_description)/urdf/accessories/sensor_arch.urdf.xacro"/>
+  <xacro:include filename="husky_mod/decorations.urdf.xacro" />
+  <xacro:include filename="husky_mod/wheel.urdf.xacro" />
+  <xacro:include filename="husky_mod/accessories/intel_realsense.urdf.xacro"/>
+  <xacro:include filename="husky_mod/accessories/sick_lms1xx_mount.urdf.xacro"/>
+  <xacro:include filename="husky_mod/accessories/sensor_arch.urdf.xacro"/>
   <xacro:property name="M_PI" value="3.14159"/>
   <xacro:macro name="husky" params="prefix">
@@ -37,5 +57,5 @@
         <origin xyz="0 0 0" rpy="0 0 0" />
         <geometry>
-          <mesh filename="package://husky_description/meshes/base_link.dae" />
+          <mesh filename="${_mesh_proto_pkg_prefix}/meshes/base_link.dae" />
         </geometry>
       </visual>
