Commit message: Re-coded in a more generic way, to avoid repeating patterns of similar URDF blocks (one block for each different depth camera for a multi-camera configuration), by using new lower-level macros defined in new library files (../lib_util_depth_cam_spawn.urdf.xacro & ./custom_part_sensor_depth_single.urdf.xacro), and with added alternative depths cameras Realsense & Zed (on top of existing Kinect). Note: this .xacro library should be generic enough to be moved down (and out) of ranger_xarm6/ sub-directory - except for <property> declarations for "ctrl_box_(width|length|height)", "cam_(front|right)_offset_[xy]" & "cam_any_offset_z", which will need to be specific to each particular robot base + arm combination.

File: urdf/ranger_xarm6/custom_part_sensor_depth.urdf.xacro (robot description, xacro)
@@ -1,4 +1,6 @@
 <?xml version="1.0"?>
 <robot xmlns:xacro="http://ros.org/wiki/xacro">
+  <xacro:include filename="../lib_util_depth_cam_spawn.urdf.xacro" />
+  <xacro:include filename="custom_part_sensor_depth_single.urdf.xacro" />
   <xacro:arg name="pkg_for_cam" default="open_vico_cameras" />
   <xacro:property name="_pkg_for_cam" default="$(arg pkg_for_cam)" />
@@ -6,7 +8,7 @@
   <xacro:property name="_pkg_loc_camera_depth"
       value="$(arg pkg_loc_camera_depth)" />
-  <xacro:property name="_use_openvico_kinect"
+  <xacro:property name="_use_openvico"
       value="${_pkg_for_cam == 'open_vico_cameras'}" />
-  <xacro:arg name="camera_model" default="kinect" />
+  <xacro:arg name="camera_model" default="zed" />
   <!--
     # Macro calls for realsense and zed (from open_vico_cameras) not yet added
@@ -14,6 +16,6 @@
   -->
 <!--
+  <xacro:arg name="camera_model" default="kinect" />
   <xacro:arg name="camera_model" default="realsense" />
-  <xacro:arg name="camera_model" default="zed" />
 -->
   <xacro:property name="_camera_model" value="$(arg camera_model)" />
@@ -53,74 +55,34 @@
   </xacro:unless>
   <!-- Control Box Properties -->
-  <xacro:property name="ctrl_box_width" value="0.27" />
-  <xacro:property name="ctrl_box_length" value="0.23" />
-  <xacro:property name="ctrl_box_height" value="0.175" />
-  <xacro:property name="cam_front_offset_x" value="0.13" />
-<!--
-  <xacro:property name="cam_front_offset_x" value="0.12" />
-  <xacro:property name="cam_front_offset_x" value="0.15" />
--->
-  <xacro:property name="cam_front_offset_y" value="0.01" />
-  <xacro:property name="cam_right_offset_x" value="-${ctrl_box_length / 2.0}" />
-  <xacro:property name="cam_right_offset_y" value="0.01" />
-<!--
-  <xacro:property name="cam_right_offset_y" value="0.1" />
--->
-  <xacro:property name="cam_any_offset_z" value="0.1" />
-  <xacro:if value="${True}">
-    <link name="realsense_mount_front"/>
-    <joint name="realsense_mount_front_joint" type="fixed">
-      <origin xyz="${ctrl_box_width / 2.0 + cam_front_offset_x}
-        ${ctrl_box_length / 2.0 + cam_front_offset_y}
-        ${ctrl_box_height / 2.0 + cam_any_offset_z}" rpy="0 0 0" />
-      <parent link="${_parent_link_for_sensor}"/>
-      <child link="realsense_mount_front" />
-    </joint>
-    <xacro:if value="${_use_openvico_kinect}">
-      <xacro:microsoft_kinect2 camera_name_prefix="camera1"
-          parent="realsense_mount_front">
-        <origin xyz="0.0115 0 0.0100" rpy="0 0 0" />
-      </xacro:microsoft_kinect2>
-    </xacro:if>
-    <xacro:unless value="${_use_openvico_kinect}">
-      <xacro:if value="${_is_kinetic}">
-        <xacro:intel_realsense_mount prefix="camera1" topic="realsense_front"
-          parent_link="realsense_mount_front"/>
-      </xacro:if>
-      <xacro:unless value="${_is_kinetic}">
-        <xacro:realsense_sensor prefix="camera1" topic="realsense_front"
-            parent="realsense_mount_front" include="0">
-          <origin xyz="0.0115 0 0.0100" rpy="0 0 0" />
-        </xacro:realsense_sensor>
-      </xacro:unless>
-    </xacro:unless>
-  </xacro:if>
-  <xacro:if value="${True}">
-    <link name="realsense_mount_right"/>
-    <joint name="realsense_mount_right_joint" type="fixed">
-      <origin xyz="${cam_right_offset_x}
-        ${(ctrl_box_length / 2.0 + cam_right_offset_y) * -1.0}
-        ${ctrl_box_height / 2.0 + cam_any_offset_z}" rpy="0 0 -1.570796" />
-      <parent link="${_parent_link_for_sensor}"/>
-      <child link="realsense_mount_right" />
-    </joint>
-    <xacro:if value="${_use_openvico_kinect}">
-      <xacro:microsoft_kinect2 camera_name_prefix="camera2"
-          parent="realsense_mount_right">
-        <origin xyz="0.0115 0 0.0100" rpy="0 0 0" />
-      </xacro:microsoft_kinect2>
-    </xacro:if>
-    <xacro:unless value="${_use_openvico_kinect}">
-      <xacro:if value="${_is_kinetic}">
-        <xacro:intel_realsense_mount prefix="camera2" topic="realsense_right"
-          parent_link="realsense_mount_right"/>
-      </xacro:if>
-      <xacro:unless value="${_is_kinetic}">
-        <xacro:realsense_sensor prefix="camera2" topic="realsense_right"
-            parent="realsense_mount_right" include="0">
-          <origin xyz="0.0115 0 0.0100" rpy="0 0 0" />
-        </xacro:realsense_sensor>
-      </xacro:unless>
-    </xacro:unless>
-  </xacro:if>
+  <xacro:arg name="ctrl_box_width" default="0.19" />
+  <xacro:arg name="ctrl_box_length" default="0.23" />
+  <xacro:arg name="ctrl_box_height" default="0.175" />
+  <xacro:property name="_ctrl_box_width" value="$(arg ctrl_box_width)" />
+  <xacro:property name="_ctrl_box_length" value="$(arg ctrl_box_length)" />
+  <xacro:property name="_ctrl_box_height" value="$(arg ctrl_box_height)" />
+  <xacro:arg name="cam_front_offset_x" default="0.13" />
+  <xacro:arg name="cam_front_offset_y" default="0.01" />
+  <xacro:property name="_cam_front_offset_x" value="$(arg cam_front_offset_x)"
+    />
+  <xacro:property name="_cam_front_offset_y" value="$(arg cam_front_offset_x)"
+    />
+  <xacro:arg name="cam_right_offset_x" default="-${_ctrl_box_length / 2.0}" />
+  <xacro:arg name="cam_right_offset_y" default="0.01" />
+  <xacro:property name="_cam_right_offset_x" value="$(arg cam_right_offset_x)"
+    />
+  <xacro:property name="_cam_right_offset_y" value="$(arg cam_right_offset_y)"
+    />
+  <xacro:arg name="cam_any_offset_z" default="0.1" />
+  <xacro:property name="_cam_any_offset_z" value="$(arg cam_any_offset_z)" />
+  <xacro:include filename="../cfg_cam_mount_map.xacro" />
+  <xacro:property name="_cam_mount_point_origin_map"
+    value="${_cam_mount_map.get( 'mount_points')}" />
+  <xacro:spawn_all_cam
+    parent_link="${_parent_link_for_sensor}"
+    camera_model="${_camera_model}"
+    use_openvico="${_use_openvico}"
+    is_kinetic="${_is_kinetic}"
+    kv_pairs="${list( _cam_mount_point_origin_map.items())}"
+    explicit_on="${dict( [ ('front', True), ('right', True) ])}"
+  />
 </robot>
